File: project_02/eagle/EtchASketch.brd (EAGLE design)
At the start: 106.7 x 81.3 mm, 20 parts, among them J1 SPI_SCREEN, J2 USB_HOST, SW1 BUTTON, SW2 BUTTON, U1 POCKETBEAGLE

Commit message: Add project
Connections:
- net BUTTON_1: now also U1.P2_22; no longer U1.P1_33
- net BUTTON_2: now also U1.P2_18; no longer U1.P1_31
- net GND: no longer U1.P1_15
- net LED_BLUE: now also U1.P2_24; no longer U1.P2_08
- net LED_GREEN: now also U1.P2_19; no longer U1.P2_20
- net LED_RED: now also U1.P1_20; no longer U1.P2_17
Routing:
- net GND: track 237.0 -> 284.5 mm
- net BUTTON_2: track 119.0 -> 75.6 mm
- net VDD_5V: track 74.3 -> 102.0 mm
- net BUTTON_1: track 82.4 -> 60.4 mm
- net LED_RED: track 53.5 -> 74.4 mm, vias 0 -> 1
- net LED_BLUE: track 46.4 -> 66.8 mm
- net AGND: track 105.7 -> 90.1 mm
- net VDD_1P8V: track 112.4 -> 100.3 mm
- net CGND: track 273.9 -> 261.9 mm, vias 1 -> 0
- net VDD_3P3V: track 144.5 -> 133.0 mm
- net CS: track 61.6 -> 68.8 mm
- net RST: track 69.8 -> 75.7 mm
- net DC: track 66.1 -> 69.7 mm, vias 0 -> 1
- net POT_LEFT: track 42.2 -> 40.4 mm
- net DM: track 51.9 -> 50.4 mm
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