File: project_02/eagle/EtchASketch.sch (EAGLE design)
At the start: 20 parts, among them J1 SPI_SCREEN, J2 USB_HOST, SW1 BUTTON, SW2 BUTTON, U1 POCKETBEAGLE

Commit message: Add project
Connections:
- net BUTTON_1: now also U1.GPIO46; no longer U1.PRU0.1
- net BUTTON_2: now also U1.GPIO47; no longer U1.PRU0.4
- net GND: no longer U1.GND@1, U1.GND@4, U1.GND@5
- net LED_BLUE: now also U1.GPIO44; no longer U1.GPIO60
- net LED_GREEN: now also U1.GPIO27; no longer U1.GPIO64
- net LED_RED: now also U1.GPIO20; no longer U1.GPIO65
Changed lines of the file:
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@@
 <net name="GND" class="0">
 <segment>
-<pinref part="U1" gate="G$1" pin="GND@4"/>
 <pinref part="GND4" gate="1" pin="GND"/>
-<wire x1="109.22" y1="170.18" x2="121.92" y2="170.18" width="0.1524" layer="91"/>
 <pinref part="U1" gate="G$1" pin="GND@2"/>
 <wire x1="109.22" y1="172.72" x2="121.92" y2="172.72" width="0.1524" layer="91"/>
 <wire x1="121.92" y1="172.72" x2="121.92" y2="170.18" width="0.1524" layer="91"/>
-<junction x="121.92" y="170.18"/>
-</segment>
-<segment>
-<pinref part="U1" gate="G$1" pin="GND@1"/>
+</segment>
+<segment>
 <pinref part="GND3" gate="1" pin="GND"/>
-<wire x1="48.26" y1="114.3" x2="38.1" y2="114.3" width="0.1524" layer="91"/>
 <pinref part="U1" gate="G$1" pin="USB1.ID"/>
 <wire x1="48.26" y1="116.84" x2="38.1" y2="116.84" width="0.1524" layer="91"/>
 <wire x1="38.1" y1="116.84" x2="38.1" y2="114.3" width="0.1524" layer="91"/>
-<junction x="38.1" y="114.3"/>
-</segment>
-<segment>
-<pinref part="U1" gate="G$1" pin="GND@5"/>
+</segment>
+<segment>
 <pinref part="GND2" gate="1" pin="GND"/>
-<wire x1="48.26" y1="170.18" x2="33.02" y2="170.18" width="0.1524" layer="91"/>
 <pinref part="U1" gate="G$1" pin="GND@3"/>
 <wire x1="48.26" y1="172.72" x2="33.02" y2="172.72" width="0.1524" layer="91"/>
 <wire x1="33.02" y1="172.72" x2="33.02" y2="170.18" width="0.1524" layer="91"/>
-<junction x="33.02" y="170.18"/>
 </segment>
 <segment>
@@
 <net name="LED_BLUE" class="0">
 <segment>
-<pinref part="U1" gate="G$1" pin="GPIO60"/>
-<wire x1="109.22" y1="119.38" x2="127" y2="119.38" width="0.1524" layer="91"/>
-<label x="121.92" y="119.38" size="1.778" layer="95"/>
-</segment>
-<segment>
 <wire x1="325.12" y1="114.3" x2="309.88" y2="114.3" width="0.1524" layer="91"/>
 <label x="309.88" y="114.3" size="1.778" layer="95"/>
 <pinref part="D3" gate="G$1" pin="ANODE"/>
 </segment>
+<segment>
+<pinref part="U1" gate="G$1" pin="GPIO44"/>
+<wire x1="109.22" y1="137.16" x2="127" y2="137.16" width="0.1524" layer="91"/>
+<label x="121.92" y="137.16" size="1.778" layer="95"/>
+</segment>
 </net>
 <net name="LED_RED" class="0">
-<segment>
-<pinref part="U1" gate="G$1" pin="GPIO65"/>
-<wire x1="109.22" y1="114.3" x2="127" y2="114.3" width="0.1524" layer="91"/>
-<label x="121.92" y="114.3" size="1.778" layer="95"/>
-</segment>
 <segment>
 <wire x1="325.12" y1="149.86" x2="309.88" y2="149.86" width="0.1524" layer="91"/>
@@
 <pinref part="D1" gate="G$1" pin="ANODE"/>
 </segment>
+<segment>
+<pinref part="U1" gate="G$1" pin="GPIO20"/>
+<wire x1="109.22" y1="142.24" x2="127" y2="142.24" width="0.1524" layer="91"/>
+<label x="121.92" y="142.24" size="1.778" layer="95"/>
+</segment>
 </net>
 <net name="LED_GREEN" class="0">
-<segment>
-<pinref part="U1" gate="G$1" pin="GPIO64"/>
-<wire x1="109.22" y1="116.84" x2="127" y2="116.84" width="0.1524" layer="91"/>
-<label x="121.92" y="116.84" size="1.778" layer="95"/>
-</segment>
 <segment>
 <wire x1="325.12" y1="132.08" x2="309.88" y2="132.08" width="0.1524" layer="91"/>
 <label x="309.88" y="132.08" size="1.778" layer="95"/>
 <pinref part="D2" gate="G$1" pin="ANODE"/>
+</segment>
+<segment>
+<pinref part="U1" gate="G$1" pin="GPIO27"/>
+<wire x1="109.22" y1="139.7" x2="127" y2="139.7" width="0.1524" layer="91"/>
+<label x="121.92" y="139.7" size="1.778" layer="95"/>
 </segment>
 </net>
@@
 </net>
 <net name="BUTTON_1" class="0">
-<segment>
-<pinref part="U1" gate="G$1" pin="PRU0.1"/>
-<wire x1="109.22" y1="101.6" x2="127" y2="101.6" width="0.1524" layer="91"/>
-<label x="121.92" y="101.6" size="1.778" layer="95"/>
-</segment>
 <segment>
 <pinref part="R3" gate="G$1" pin="2"/>
@@
 <pinref part="SW1" gate="G$1" pin="3"/>
 </segment>
+<segment>
+<pinref part="U1" gate="G$1" pin="GPIO46"/>
+<wire x1="109.22" y1="134.62" x2="127" y2="134.62" width="0.1524" layer="91"/>
+<label x="121.92" y="134.62" size="1.778" layer="95"/>
+</segment>
 </net>
 <net name="BUTTON_2" class="0">
@@
 </segment>
 <segment>
-<pinref part="U1" gate="G$1" pin="PRU0.4"/>
-<wire x1="109.22" y1="93.98" x2="127" y2="93.98" width="0.1524" layer="91"/>
-<label x="121.92" y="93.98" size="1.778" layer="95"/>
-</segment>
-</net>
+<pinref part="U1" gate="G$1" pin="GPIO47"/>
+<wire x1="109.22" y1="132.08" x2="127" y2="132.08" width="0.1524" layer="91"/>
+<label x="121.92" y="132.08" size="1.778" layer="95"/>
+</segment>
+</net>
